File: KiCad/Stormbreaker.kicad_pcb (KiCad board)
At the start: 4 copper layers, 50.2 x 21.5 mm, 49 parts, among them J1 Micro_SD_Card_Det2, J2 USB_C_Receptacle_USB2.0_14P, J3 PROG, J5 I2C, Q1 PMOS, Q2 NMOS, SW1 SW_Push, U1 BQ25895RTW, U3 ATtiny1616-M, U4 HUSB238A

Commit message: Add fancy logo
Other:
- board text added: "STORMBREAKER"

Commit message: Misc changes, README.md update
Parts:
- C5, C6: value 10uF -> 22uF
- J1: value Micro_SD_Card_Det2 -> Micro_SD_Card_Det1
Connections:
- J1 pad 10: SD_DECT -> GND
- J1 pad 9: GND -> SD_DECT
Routing:
- net SD_DECT: track 14.1 -> 13.7 mm, vias 2 -> 0

Commit message: Minor hardware changes
Parts:
- TP3: value 3V3 -> 3.3V
- moved C14 0.25 mm to (145.0, 49.8)
- moved R8 0.25 mm to (138.8, 51.3)
Routing:
- net Net-(Q1-G): track 26.2 -> 25.3 mm
- net VCC: track 8.51 -> 8.26 mm, vias 57 -> 71
- net GND: vias 41 -> 50
- net /BATT: vias 19 -> 28
Other:
- board text added: "-"
- board text added: "@VoxelTek 2025"
- board text added: "p"
