File: KiCad/Stormbreaker.kicad_pcb (KiCad board)
At the start: 4 copper layers, 50.2 x 21.5 mm, 49 parts, among them J1 Micro_SD_Card_Det1, J2 USB_C_Receptacle_USB2.0_14P, J3 PROG, J5 I2C, Q1 PMOS, Q2 NMOS, SW1 SW_Push, U1 BQ25895RTW, U3 ATtiny1616-M, U4 HUSB238A

Commit message: Generate ibom, add value for GL835
Parts:
- TP3: value 3.3V -> 3V3
- U2: value ~ -> GL835
