File: KiCad/Stormbreaker.kicad_sch (KiCad schematic)
At the start: 49 parts, among them J1 Micro_SD_Card_Det2, J2 USB_C_Receptacle_USB2.0_14P, J3 PROG, J5 I2C, Q1 PMOS, Q2 NMOS, SW1 SW_Push, U1 BQ25895RTW, U3 ATtiny1616-M, U4 HUSB238A

Commit message: Misc board improvements
Parts:
- removed C11: 4.7μF, Capacitor_SMD:C_0603_1608Metric, symbol Device:C_Small
Connections:
- net BQ_~{INT}: now reaches U1.7 (INT)
- net BQ_~{INT}: now also U3.15 (PC0)
- net BQ_STAT: no longer names the net of U1.4 (STAT)
- net BQ_STAT: no longer U3.15 (PC0)
Changed lines of the file:
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@@
 	)
 	(junction
-		(at 133.35 154.94)
-		(diameter 0)
-		(color 0 0 0 0)
-	)
-	(junction
 		(at 62.23 156.21)
 		(diameter 0)
@@
 	)
 	(no_connect
+		(at 76.2 83.82)
+	)
+	(no_connect
 		(at 76.2 71.12)
 	)
@@
 	)
 	(no_connect
-		(at 76.2 93.98)
-	)
-	(no_connect
 		(at 187.96 85.09)
 	)
@@
 	(wire
 		(pts
-			(xy 133.35 154.94) (xy 135.89 154.94)
+			(xy 113.03 154.94) (xy 135.89 154.94)
 		)
 		(stroke
@@
 	(wire
 		(pts
-			(xy 113.03 154.94) (xy 133.35 154.94)
-		)
-		(stroke
-			(width 0)
-			(type default)
-		)
-	)
-	(wire
-		(pts
 			(xy 187.96 74.93) (xy 207.01 74.93)
 		)
@@
 	(wire
 		(pts
-			(xy 59.69 83.82) (xy 76.2 83.82)
-		)
-		(stroke
-			(width 0)
-			(type default)
-		)
-	)
-	(wire
-		(pts
 			(xy 134.62 66.04) (xy 113.03 66.04)
 		)
@@
 	(wire
 		(pts
-			(xy 133.35 154.94) (xy 133.35 156.21)
+			(xy 59.69 93.98) (xy 76.2 93.98)
 		)
 		(stroke
@@
 		)
 	)
-	(label "BQ_STAT"
-		(at 59.69 83.82 0)
-		(effects
-			(font
-				(size 1.27 1.27)
-			)
-			(justify left bottom)
-		)
-	)
-	(label "BQ_STAT"
-		(at 147.32 92.71 0)
+	(label "BQ_~{INT}"
+		(at 59.69 93.98 0)
 		(effects
 			(font
@@
 		)
 	)
+	(label "BQ_~{INT}"
+		(at 147.32 92.71 0)
+		(effects
+			(font
+				(size 1.27 1.27)
+			)
+			(justify left bottom)
+		)
+	)
 	(label "PowerButton"
 		(at 219.71 74.93 180)
@@
 	)
 	(symbol
-		(lib_id "Device:C_Small")
-		(at 133.35 158.75 0)
-		(unit 1)
-		(exclude_from_sim no)
-		(in_bom yes)
-		(on_board yes)
-		(dnp no)
-		(property "Reference" "C11"
-			(at 135.89 158.242 0)
-			(effects
-				(font
-					(size 1.27 1.27)
-				)
-				(justify left)
-			)
-		)
-		(property "Value" "4.7μF"
-			(at 135.89 160.782 0)
-			(effects
-				(font
-					(size 1.27 1.27)
-				)
-				(justify left)
-			)
-		)
-		(property "Footprint" "Capacitor_SMD:C_0603_1608Metric"
-			(at 133.35 158.75 0)
-			(effects
-				(font
-					(size 1.27 1.27)
-				)
-				(hide yes)
-			)
-		)
-		(property "Datasheet" "~"
-			(at 133.35 158.75 0)
-			(effects
-				(font
-					(size 1.27 1.27)
-				)
-				(hide yes)
-			)
-		)
-		(property "Description" "Unpolarized capacitor, small symbol"
-			(at 133.35 158.75 0)
-			(effects
-				(font
-					(size 1.27 1.27)
-				)
-				(hide yes)
-			)
-		)
-		(pin "1"
-		)
-		(pin "2"
-		)
-		(instances
-			(project "Stormbreaker"
-				(path "/dcc89f95-4ae4-4756-aa81-33bf4d3c86ca"
-					(reference "C11")
-					(unit 1)
-				)
-			)
-		)
-	)
-	(symbol
 		(lib_id "Connector:TestPoint")
 		(at 59.69 176.53 0)
@@
 					(unit 1)
 				)
-			)
-		)
-	)
-	(symbol
-		(lib_id "power:GND")
-		(at 133.35 161.29 0)
-		(unit 1)
-		(exclude_from_sim no)
-		(in_bom yes)
-		(on_board yes)
-		(dnp no)
-		(fields_autoplaced yes)
-		(property "Reference" "#PWR015"
-			(at 133.35 167.64 0)
-			(effects
-				(font
-					(size 1.27 1.27)
-				)
-				(hide yes)
-			)
-		)
-		(property "Value" "GND"
-			(at 133.35 166.37 0)
-			(effects
-				(font
-					(size 1.27 1.27)
-				)
-			)
-		)
-		(property "Footprint" ""
-			(at 133.35 161.29 0)
-			(effects
-				(font
-					(size 1.27 1.27)
-				)
-				(hide yes)
-			)
-		)
-		(property "Datasheet" ""
-			(at 133.35 161.29 0)
-			(effects
-				(font
-					(size 1.27 1.27)
-				)
-				(hide yes)
-			)
-		)
-		(property "Description" "Power symbol creates a global label with name \"GND\" , ground"
-			(at 133.35 161.29 0)
-			(effects
-				(font
-					(size 1.27 1.27)
-				)
-				(hide yes)
-			)
-		)
-		(pin "1"
-		)
-		(instances
-			(project "Stormbreaker"
-				(path "/dcc89f95-4ae4-4756-aa81-33bf4d3c86ca"
-					(reference "#PWR015")
-					(unit 1)
-				)

Commit message: v3 hardware design: largely complete
Parts:
- removed R12: 6.04k, Resistor_SMD:R_0402_1005Metric, symbol Device:R_Small
- added TP9: GND, TestPoint:TestPoint_Pad_D2.5mm, symbol Connector:TestPoint
- C12: footprint Capacitor_SMD:C_0603_1608Metric -> Capacitor_SMD:C_0402_1005Metric
- C5, C6: value 10uF -> 22uF
- SW1: footprint Button_Switch_SMD:SW_Push_1P1T-MP_NO_Horizontal_Alps_SKRTLAE010 -> Stormbreaker:SW_TL3330AF260QG; Digikey (none) -> https://www.digikey.com.au/en/products/detail/e-switch/TL33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; Mouser https://www.digikey.com.au/en/products/detail/alps-alpine/S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 -> (none)
- TP10, TP11: footprint Stormbreaker:TestPoint_Pad_D0.75mm_Small -> Stormbreaker:TestPoint_Pad_D1.0mm_Small
- TP4: footprint TestPoint:TestPoint_Pad_D1.0mm -> Stormbreaker:TestPoint_Pad_D1.0mm_Small
Connections:
- net GND: now also R6.1, U4.8 (ADDR), TP9.1
- net SCL_2: now also U4.10 (SCL)
- net SDA_2: now also U4.9 (SDA)
- net VBUS: no longer R6.1
- no-connect marks 22 -> 20
Other:
- moved on the sheet: C15, R11, R6, U4

Commit message: Misc changes, README.md update
Parts:
- removed J1: Micro_SD_Card_Det2, Connector_Card:microSD_HC_Hirose_DM3D-SF, symbol Connector:Micro_SD_Card_Det2
- added J1: Micro_SD_Card_Det1, Connector_Card:microSD_HC_Hirose_DM3D-SF, symbol Connector:Micro_SD_Card_Det1
Connections:
- net GND: now also J1.10 (SHIELD), J1.11 (SHIELD), J1.6 (VSS)
- net SD_CLK: now also J1.5 (CLK)
- net SD_CMD: now also J1.3 (CMD)
- net SD_D0: now also J1.7 (DAT0)
- net SD_D1: now also J1.8 (DAT1)
- net SD_D2: now also J1.1 (DAT2)
- net SD_D3: now also J1.2 (DAT3/CD)
- net SD_DECT: now also J1.9 (DET)
- net SD_VCC: now also J1.4 (VDD)
Changed lines of the file:
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@@
 		(color 0 0 0 0)
 	)
-	(junction
-		(at 217.17 137.16)
-		(diameter 0)
-		(color 0 0 0 0)
-	)
 	(no_connect
 		(at 76.2 96.52)
@@
 	(wire
 		(pts
-			(xy 217.17 137.16) (xy 229.87 137.16)
-		)
-		(stroke
-			(width 0)
-			(type default)
-		)
-	)
-	(wire
-		(pts
 			(xy 146.05 90.17) (xy 146.05 91.44)
 		)
@@
 	(wire
 		(pts
-			(xy 217.17 137.16) (xy 217.17 140.97)
+			(xy 217.17 127) (xy 217.17 140.97)
 		)
 		(stroke
@@
 	(wire
 		(pts
-			(xy 217.17 127) (xy 217.17 137.16)
-		)
-		(stroke
-			(width 0)
-			(type default)
-		)
-	)
-	(wire
-		(pts
 			(xy 134.62 66.04) (xy 113.03 66.04)
 		)
@@
 	(global_label "SD_DECT"
 		(shape output)
-		(at 229.87 134.62 180)
+		(at 229.87 137.16 180)
 		(fields_autoplaced yes)
 		(effects
@@
 		)
 		(property "Intersheetrefs" "${INTERSHEET_REFS}"
-			(at 218.7811 134.62 0)
+			(at 218.7811 137.16 0)
 			(effects
 				(font
@@
 	)
 	(symbol
+		(lib_id "Connector:Micro_SD_Card_Det1")
+		(at 252.73 124.46 0)
+		(unit 1)
+		(exclude_from_sim no)
+		(in_bom yes)
+		(on_board yes)
+		(dnp no)
+		(fields_autoplaced yes)
+		(property "Reference" "J1"
+			(at 253.365 102.87 0)
+			(effects
+				(font
+					(size 1.27 1.27)
+				)
+			)
+		)
+		(property "Value" "Micro_SD_Card_Det1"
+			(at 253.365 105.41 0)
+			(effects
+				(font
+					(size 1.27 1.27)
+				)
+			)
+		)
+		(property "Footprint" "Connector_Card:microSD_HC_Hirose_DM3D-SF"
+			(at 304.8 106.68 0)
+			(effects
+				(font
+					(size 1.27 1.27)
+				)
+				(hide yes)
+			)
+		)
+		(property "Datasheet" "https://www.hirose.com/en/product/document?clcode=&productname=&series=DM3&documenttype=Catalog&lang=en&documentid=D49662_en"
+			(at 252.73 121.92 0)
+			(effects
+				(font
+					(size 1.27 1.27)
+				)
+				(hide yes)
+			)
+		)
+		(property "Description" "Micro SD Card Socket with one card detection pin"
+			(at 252.73 124.46 0)
+			(effects
+				(font
+					(size 1.27 1.27)
+				)
+				(hide yes)
+			)
+		)
+		(property "Model" "DM3D-SF(41)"
+			(at 252.73 124.46 0)
+			(effects
+				(font
+					(size 1.27 1.27)
+				)
+				(hide yes)
+			)
+		)
+		(pin "3"
+		)
+		(pin "2"
+		)
+		(pin "4"
+		)
+		(pin "5"
+		)
+		(pin "6"
+		)
+		(pin "7"
+		)
+		(pin "10"
+		)
+		(pin "9"
+		)
+		(pin "8"
+		)
+		(pin "1"
+		)
+		(pin "11"
+		)
+		(instances
+			(project ""
+				(path "/dcc89f95-4ae4-4756-aa81-33bf4d3c86ca"
+					(reference "J1")
+					(unit 1)
+				)
+			)
+		)
+	)
+	(symbol
 		(lib_id "Device:C_Small")
 		(at 43.18 41.91 180)
@@
 					(unit 1)
 				)
-			)
-		)
-	)
-	(symbol
-		(lib_id "Connector:Micro_SD_Card_Det2")
-		(at 252.73 124.46 0)
-		(unit 1)
-		(exclude_from_sim no)
-		(in_bom yes)
-		(on_board yes)
-		(dnp no)
-		(fields_autoplaced yes)
-		(property "Reference" "J1"
-			(at 253.365 102.87 0)
-			(effects
-				(font
-					(size 1.27 1.27)
-				)
-			)
-		)
-		(property "Value" "Micro_SD_Card_Det2"
-			(at 253.365 105.41 0)
-			(effects
-				(font
-					(size 1.27 1.27)
-				)
-			)
-		)
-		(property "Footprint" "Connector_Card:microSD_HC_Hirose_DM3D-SF"
-			(at 304.8 106.68 0)
-			(effects
-				(font
-					(size 1.27 1.27)
-				)
-				(hide yes)
-			)
-		)
-		(property "Datasheet" "https://www.hirose.com/en/product/document?clcode=&productname=&series=DM3&documenttype=Catalog&lang=en&documentid=D49662_en"
-			(at 255.27 121.92 0)
-			(effects
-				(font
-					(size 1.27 1.27)
-				)
-				(hide yes)
-			)
-		)
-		(property "Description" "Micro SD Card Socket with two card detection pins"
-			(at 252.73 124.46 0)
-			(effects
-				(font
-					(size 1.27 1.27)
-				)
-				(hide yes)
-			)
-		)
-		(property "Model" "DM3D-SF(41)"
-			(at 252.73 124.46 0)
-			(effects
-				(font
-					(size 1.27 1.27)
-				)
-				(hide yes)
-			)
-		)
-		(pin "2"
-		)
-		(pin "1"
-		)
-		(pin "3"
-		)
-		(pin "4"
-		)
-		(pin "7"
-		)
-		(pin "8"
-		)
-		(pin "9"
-		)
-		(pin "10"
-		)
-		(pin "5"
-		)
-		(pin "6"
-		)
-		(pin "11"
-		)
-		(instances
-			(project ""
-				(path "/dcc89f95-4ae4-4756-aa81-33bf4d3c86ca"
-					(reference "J1")
-					(unit 1)
-				)

Commit message: Generate ibom, add value for GL835
Parts:
- U2: value ~ -> GL835
Changed lines of the file:
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@@
 		(fields_autoplaced yes)
 		(property "Reference" "U2"
-			(at 96.52 146.05 0)
+			(at 96.52 144.78 0)
 			(effects
 				(font
@@
 			)
 		)
-		(property "Value" "~"
-			(at 96.52 148.59 0)
+		(property "Value" "GL835"
+			(at 96.52 147.32 0)
 			(effects
 				(font
